File: tac5212.kicad_sch (KiCad schematic)
At the start: 49 parts, among them J1 DIGI, J2 AIN, J3 AOUT, J4 DIN, J5 VDC, J6 Qwiic, J8 CLK, U1 XTAC5212IRGER, U2 SPX3819M5-L-3-3, Y1 830207659209

Commit message: v1.0 sent to fab - added AVDD supply
Parts:
- removed H1: MH, MountingHole:MountingHole_2.2mm_M2, symbol Mechanical:MountingHole
- removed J2: AIN, Connector_PinHeader_2.54mm:PinHeader_1x06_P2.54mm_Vertical, symbol Connector_Generic:Conn_01x06
- removed J3: AOUT, Connector_PinHeader_2.54mm:PinHeader_1x06_P2.54mm_Vertical, symbol Connector_Generic:Conn_01x06
- added C18: 0.1uF, Capacitor_SMD:C_0805_2012Metric, symbol Device:C_Small
- added J10: AIN_GND, Connector_PinHeader_2.54mm:PinHeader_1x02_P2.54mm_Vertical, symbol Connector_Generic:Conn_01x02
- added J11: AOUT1, Connector_PinHeader_2.54mm:PinHeader_1x02_P2.54mm_Vertical, symbol Connector_Generic:Conn_01x02
- added J12: AOUT2, Connector_PinHeader_2.54mm:PinHeader_1x02_P2.54mm_Vertical, symbol Connector_Generic:Conn_01x02
- added J13: 54-00178, Headphone_Jack:TENSILITY_54-00178, symbol Headphone_Jack:54-00178
- added J2: AIN1, Connector_PinHeader_2.54mm:PinHeader_1x02_P2.54mm_Vertical, symbol Connector_Generic:Conn_01x02
- added J3: AOUT_GND, Connector_PinHeader_2.54mm:PinHeader_1x02_P2.54mm_Vertical, symbol Connector_Generic:Conn_01x02
- added J7: MIC_GND, Connector_PinHeader_2.54mm:PinHeader_1x01_P2.54mm_Vertical, symbol Connector_Generic:Conn_01x01
- added J9: AIN2, Connector_PinHeader_2.54mm:PinHeader_1x02_P2.54mm_Vertical, symbol Connector_Generic:Conn_01x02
- added JP10: Jumper_2_Small_Open, Jumper:SolderJumper-2_P1.3mm_Open_TrianglePad1.0x1.5mm, symbol Jumper:Jumper_2_Small_Open
- added TP5: AVDD, TestPoint:TestPoint_THTPad_D1.0mm_Drill0.5mm, symbol Connector:TestPoint
- added U3: SPX3819M5-L-3-3, Package_TO_SOT_SMD:SOT-23-5, symbol Regulator_Linear:SPX3819M5-L-3-3
- TP3: value 3V3 -> IOVDD; footprint TestPoint:TestPoint_Pad_D1.0mm -> TestPoint:TestPoint_THTPad_D1.0mm_Drill0.5mm
Connections:
- net +3.3V: now also JP10.2 (B); no longer C1.1, C2.1, R1.1, U1.23 (AVDD)
- net CIN1N: now also J2.2 (Pin_2)
- net CIN1P: now also J2.1 (Pin_1)
- net CIN2N: now also J9.2 (Pin_2)
- net CIN2P: now also J9.1 (Pin_1)
- net COUT1N: now also J11.1 (Pin_1)
- net COUT1P: now also J11.2 (Pin_2), J13.4
- net COUT2N: now also J12.2 (Pin_2)
- net COUT2P: now also J12.1 (Pin_1), J13.3
- net GND: now also C18.2, J10.1 (Pin_1), J10.2 (Pin_2), J13.1, J13.2, J3.1 (Pin_1), J3.2 (Pin_2), J7.1 (Pin_1), U3.2 (GND)
- net VDC: now also U3.1 (IN), U3.3 (EN)
- new net: C18.1, U3.4 (BP)
- new net AVDD: C1.1, C2.1, JP10.1 (A), R1.1, TP5.1, U1.23 (AVDD), U3.5 (OUT)
- no-connect marks 1 -> 3
Other:
- moved on the sheet: C1, C17, C2, C4, C5, C6, C7, H2, H3, J5, J6, R2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

Commit message: add HTML BOM
Parts:
- G1, J7, JP10, TP1, TP3, TP5: now left out of the parts list
- U1: footprint footprints:VQFN24_RGE_CORNERPADS_TEX -> VQFN24_RGE_CORNERPADS_TEX
Other:
- note added: "ANALOG"
- note added: "DIGITAL"
- note added: "MECH/TP/INDICATOR"
- note added: "POWER"
- moved on the sheet: C1, C10, C11, C12, C13, C14, C15, C16, C2, C3, C4, C5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
